File: automotive_ethernet.kicad_sch (KiCad schematic)
At the start: 11 parts, among them U12 LAN8651B1-E/LMX, Y3 25MHz

Commit message: Remove non-existent security fields from bluer characteristics
The bluer crate's CharacteristicWrite and CharacteristicNotify
don't have encrypt_*/secure_* fields - removed them.

Co-Authored-By: Claude Opus 4.5 <noreply@anthropic.com>
Parts:
- C16: footprint Capacitor_SMD:CP_Elec_3x5.3 -> Capacitor_SMD:C_0805_2012Metric
- FB1, FB2: footprint Inductor_SMD:L_0201_0603Metric -> Inductor_SMD:L_0402_1005Metric
- U12: now left out of the parts list
Changed lines of the file:
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@@
 			)
 		)
-		(property "Footprint" "Inductor_SMD:L_0201_0603Metric"
+		(property "Footprint" "Inductor_SMD:L_0402_1005Metric"
 			(at 163.83 72.898 90)
 			(effects
@@
 		(unit 1)
 		(exclude_from_sim no)
-		(in_bom yes)
+		(in_bom no)
 		(on_board yes)
 		(dnp no)
@@
 			)
 		)
-		(property "Footprint" "Capacitor_SMD:CP_Elec_3x5.3"
+		(property "Footprint" "Capacitor_SMD:C_0805_2012Metric"
 			(at 44.45 64.4652 0)
 			(effects
@@
 			)
 		)
-		(property "Footprint" "Inductor_SMD:L_0201_0603Metric"
+		(property "Footprint" "Inductor_SMD:L_0402_1005Metric"
 			(at 163.83 83.058 90)
 			(effects
