File: Perfect-Vision-ECU.kicad_pcb (KiCad board)
At the start: 2 copper layers, 92 x 92 mm, 62 parts, among them J1 ISOBUS, J11 Boot, J5 USB_C_Receptacle_USB2.0_16P, J6 Conn_Coaxial, J7 SECONDARY, J8 Reset, K1 G6K-2 12V, Q1 PZT2222A, U1 NEO-M9N-00B, U2 ESP32-S3-MINI-1, U3 LM2596S-3.3, U6 MCP2515-xSO, U7 SN65HVD230, U8 SN65HVD230, Y2 8MHz

Commit message: Fixes 20/10/2026
Parts:
- removed D5: 3.3v, Diode_SMD:D_SOD-123
- removed R16: 10k, Resistor_SMD:R_0402_1005Metric
- removed R17: 100k, Resistor_SMD:R_0402_1005Metric
- D9: footprint Diode_SMD:Nexperia_DSN1608-2_1.6x0.8mm -> Diode_SMD:D_SMA
- L1: footprint Inductor_SMD:L_7.3x7.3_H4.5 -> Inductor_SMD:L_12x12mm_H4.5mm
- moved C6 57.6 mm to (134.0, 120.0)
- moved Y2 55.9 mm to (145.5, 176.1), turned to 90 degrees
- moved C7 52.9 mm to (145.7, 179.5), turned to 0 degrees
- moved C5 47.6 mm to (148.0, 124.5)
- moved C8 40.7 mm to (145.7, 173.0), turned to 180 degrees
- moved R8 40.2 mm to (144.5, 138.5)
- moved R20 21.2 mm to (135.8, 165.0), turned to 180 degrees
- moved R7 19.5 mm to (180.0, 131.5), turned to 180 degrees
- moved U7 18.0 mm to (178.0, 135.5), turned to 0 degrees
- moved D2 6.96 mm to (185.5, 136.0)
- moved C11 6.07 mm to (171.0, 161.5)
- moved C9 3.02 mm to (171.0, 164.0)
- moved D12 1.68 mm to (168.5, 157.9)
- moved J1 1.67 mm to (114.4, 114.0)
- moved L1 1.50 mm to (157.8, 130.0)
Connections:
- net /Power/12V_Tractor renamed /Power/12V_Tractor_1
- D2 pad 1: CAN1_H_IMPL -> CAN0 H
- D2 pad 3: CAN1_L_IMPL -> CAN0 L
- D3 pad 1: CAN1 H -> CAN1_H_ECU
- D3 pad 3: CAN1 L -> CAN1_L_ECU
- K1 pad 3: CAN1_H_IMPL -> CAN1_H_ECU
- K1 pad 6: CAN1_L_IMPL -> CAN1_L_ECU
- U1 pad 14: LNA_EN -> +3.3V
- U1 pad 4: Net-(D5-K) -> unconnected-(U1-EXTINT-Pad4)
- U2 pad 34: LNA_EN -> unconnected-(U2-IO38-Pad34)
- U2 pad 39: RXD0 -> TXD0
- U2 pad 40: TXD0 -> RXD0
- U3 pad 3: unconnected-(U3-GND-Pad3) -> GND
- U7 pad 6: CAN1_L_IMPL -> CAN0 L
- U7 pad 7: CAN1_H_IMPL -> CAN0 H
- U8 pad 6: CAN1 L -> CAN1_L_ECU
- U8 pad 7: CAN1 H -> CAN1_H_ECU
Routing:
- net CAN1_H_ECU: track 0.00 -> 99.7 mm, vias 0 -> 3
- net CAN1_L_ECU: track 0.00 -> 83.0 mm, vias 0 -> 2
- net LNA_EN: track 81.3 -> 0.00 mm, vias 2 -> 0
- net CAN1_H_IMPL: track 78.3 -> 0.00 mm
- net GND: track 501.2 -> 574.9 mm, vias 0 -> 15
- net CAN1_L_IMPL: track 72.8 -> 0.00 mm
- net Net-(U6-OSC1): track 76.9 -> 7.07 mm, vias 2 -> 0
- net Net-(D5-K): track 64.9 -> 0.00 mm, vias 2 -> 0
- net Net-(U6-OSC2): track 75.0 -> 10.1 mm, vias 2 -> 0
- net CAN1 H: track 44.2 -> 0.00 mm
- net IO5: track 69.8 -> 112.4 mm, vias 2 -> 4
- net Net-(U8-Rs): track 43.8 -> 1.40 mm
- net CAN1 L: track 41.2 -> 0.00 mm
- net CAN0 L: track 9.12 -> 41.8 mm
- net CAN0 H: track 9.12 -> 39.5 mm
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Other:
- board text added: "ISOBUS"
- board text added: "SECONDARY"
