File: gps.kicad_sch (KiCad schematic)
At the start: 14 parts, among them J6 Conn_Coaxial, U1 NEO-M9N-00B

Commit message: Fixes 20/10/2026
Parts:
- removed D5: 3.3v, Diode_SMD:D_SOD-123, symbol Device:D_Zener
- removed R16: 10k, Resistor_SMD:R_0402_1005Metric, symbol Device:R
- removed R17: 100k, Resistor_SMD:R_0402_1005Metric, symbol Device:R
Connections:
- net LNA_EN is gone; now on net +3.3V: U1.14 (LNA_EN)
