File: power.kicad_sch (KiCad schematic)
At the start: 14 parts, among them J1 ISOBUS, J7 SECONDARY, U3 LM2596S-3.3

Commit message: Fixes 20/10/2026
Parts:
- D9: footprint Diode_SMD:Nexperia_DSN1608-2_1.6x0.8mm -> Diode_SMD:D_SMA
- L1: footprint Inductor_SMD:L_7.3x7.3_H4.5 -> Inductor_SMD:L_12x12mm_H4.5mm
Connections:
- net GND: now also U3.3 (GND)
- net 12V_Tractor renamed 12V_Tractor_1
Changed lines of the file:
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@@
+	)
+	(junction
+		(at 118.11 87.63)
+		(diameter 0)
+		(color 0 0 0 0)
 	)
 	(junction
@@
 	(wire
 		(pts
+			(xy 118.11 81.28) (xy 118.11 87.63)
+		)
+		(stroke
+			(width 0)
+			(type default)
+		)
+	)
+	(wire
+		(pts
 			(xy 135.89 76.2) (xy 142.24 76.2)
 		)
@@
 	(wire
 		(pts
-			(xy 101.6 87.63) (xy 135.89 87.63)
+			(xy 101.6 87.63) (xy 118.11 87.63)
 		)
 		(stroke
@@
 	(wire
 		(pts
+			(xy 118.11 87.63) (xy 135.89 87.63)
+		)
+		(stroke
+			(width 0)
+			(type default)
+		)
+	)
+	(wire
+		(pts
 			(xy 191.77 107.95) (xy 198.12 107.95)
 		)
@@
 		)
 	)
-	(label "12V_Tractor"
-		(at 148.59 107.95 0)
+	(label "12V_Tractor_1"
+		(at 90.17 107.95 0)
 		(effects
 			(font
@@
 			)
 		)
-		(property "Footprint" "Inductor_SMD:L_7.3x7.3_H4.5"
+		(property "Footprint" "Inductor_SMD:L_12x12mm_H4.5mm"
 			(at 146.05 76.2 0)
 			(effects
@@
 			)
 		)
-		(property "Footprint" "Diode_SMD:Nexperia_DSN1608-2_1.6x0.8mm"
+		(property "Footprint" "Diode_SMD:D_SMA"
 			(at 180.975 113.03 0)
 			(effects
